File: KiCAD Files/DS_to_SNES_Controller.kicad_sch (KiCad schematic)
At the start: 39 parts, among them J1 Conn_01x01_Pin, J2 Conn_01x01_Pin, J3 Conn_01x01_Pin, J4 Conn_01x01_Pin, J5 Conn_01x01_Pin, U2 4021, U3 4021, X1 Conn_01x01_Pin, Y1 Conn_01x01_Pin

Commit message: Changed total layers to 2
Parts:
- added C3, C5: 0.1uF, Capacitor_SMD:C_0603_1608Metric_Pad1.08x0.95mm_HandSolder, symbol Device:C_Small
- added C4, C6: 1uF, Capacitor_SMD:C_0603_1608Metric_Pad1.08x0.95mm_HandSolder, symbol Device:C_Small
Connections:
- net +5V: now also C1.1, C2.1, C3.1, C4.1, C5.1, C6.1
- net GND: now also C1.2, C2.2, C3.2, C4.2, C5.2, C6.2
Other:
- note added: "Buttons"
- note added: "DS to SNES Controller"
- note added: "SNES Connection"
- title: (none) -> DS to SNES Controller
- moved on the sheet: C1, C2, R1, R2, R3, RN1, RN2, U1, U2, U3
